File: pcb/macropad.kicad_pcb (KiCad board)
At the start: 2 copper layers, 20.5 x 56.7 mm, 4 parts, among them SW1 SW_Push, SW2 SW_Push, SW3 SW_Push, U1 MOUDLE-SEEEDUINO-XIAO

Commit message: Welp, fw is almost done, but I just read that only QMK, KMK and ZMK are allowed.
Routing:
- net GND: track 38.0 -> 42.2 mm
Changed lines of the file:
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@@
+	(segment
+		(start -203.265 148.005)
+		(end -204.47 146.8)
+		(width 0.2)
+		(layer "F.Cu")
+		(net "GND")
+	)
+	(segment
+		(start -204.47 146.8)
+		(end -207 146.8)
+		(width 0.2)
+		(layer "F.Cu")
+		(net "GND")
+	)
 	(segment
 		(start -203.265 148.005)
@@
 		(layer "F.Cu")
 		(net "GND")
-	)
-	(segment
-		(start -207 154.42)
-		(end -199.08 154.42)
-		(width 0.2)
-		(layer "B.Cu")
-		(net "Net-(U1-PA5_A9_D9_MISO)")
-	)
-	(segment
-		(start -196.915 156.585)
-		(end -196.915 164.42)
-		(width 0.2)
-		(layer "B.Cu")
-		(net "Net-(U1-PA5_A9_D9_MISO)")
-	)
-	(segment
-		(start -199.08 154.42)
-		(end -196.915 156.585)
-		(width 0.2)
-		(layer "B.Cu")
-		(net "Net-(U1-PA5_A9_D9_MISO)")
 	)
 	(segment
@@
 		(net "Net-(U1-PA7_A8_D8_SCK)")
 	)
+	(segment
+		(start -207 154.42)
+		(end -199.08 154.42)
+		(width 0.2)
+		(layer "B.Cu")
+		(net "Net-(U1-PA5_A9_D9_MISO)")
+	)
+	(segment
+		(start -196.915 156.585)
+		(end -196.915 164.42)
+		(width 0.2)
+		(layer "B.Cu")
+		(net "Net-(U1-PA5_A9_D9_MISO)")
+	)
+	(segment
+		(start -199.08 154.42)
+		(end -196.915 156.585)
+		(width 0.2)
+		(layer "B.Cu")
+		(net "Net-(U1-PA5_A9_D9_MISO)")
+	)
 	(embedded_fonts no)
